File: models/right_v1/top-plate-kicad/symphonie6_right.kicad_sch (KiCad schematic)
At the start: 81 parts, among them SW0_1 SW_Push, SW0_2 SW_Push, SW0_3 SW_Push, SW0_4 SW_Push, SW0_5 RotaryEncoder_Switch, SW1 SW_SPDT, SW1_0 SW_Push, SW1_2 SW_Push, SW1_3 SW_Push, SW1_4 SW_Push, SW1_5 SW_Push, SW2_0 SW_Push, SW2_1 SW_Push, SW2_3 SW_Push, SW2_4 SW_Push, SW2_5 SW_Push, SW3_0 SW_Push, SW3_1 SW_Push, SW3_2 SW_Push, SW3_4 SW_Push, SW4_0 SW_Push, SW4_1 SW_Push, SW4_2 SW_Push, SW4_3 SW_Push, SW5_0 SW_Push, SW5_1 SW_Push, SW5_2 SW_Push, SW5_3 SW_Push, SW5_4 SW_Push, SW6_0 SW_Push, SW6_1 SW_Push, SW6_2 SW_Push, SW6_3 SW_Push, SW6_4 SW_Push

Commit message: feat: added several 3D models
Parts:
- removed D44, D45: D, sym6_salicyl:Diode_TH_SMD, symbol roBa-Keyboard:D
- removed SW0_5: RotaryEncoder_Switch, KiCad_Rotary_Encoder:RotaryEncoder_Alps_EC11E-Switch_Vertical_H20mm, symbol KiCad_Rotray_Encoder:RotaryEncoder_Switch
- removed SW1_5, SW2_5: SW_Push, sym6_salicyl:Choc_v2_Hotswap_1u, symbol roBa-Keyboard:SW_Push
- added J1: ~, sym6_roba:pmw3610_connector, symbol roba:pmw3610_breakout
- added SW0_5: SW_Push, sym6_salicyl:Choc_v2_Hotswap_1u, symbol roBa-Keyboard:SW_Push
Connections:
- net 3.3V: now also J1.4 (Vin)
- net GND: now also J1.3 (GND)
- net INTR: now also D43.1 (K)
- net PIN0: now also SW0_5.2
- net PIN5: now also D42.1 (K)
- net at D41.2 (A): now also SW0_5.1
- net at D43.2 (A): now also D41.1 (K), D42.2 (A)
- net MOTION: now reaches U1.15 (NFC1_0.09)
- net MOTION: now also J1.7 (MOTION)
- net CS: now reaches U1.16 (NFC2_0.10)
- net CS: now also J1.2 (nCS)
- net RE_A1 renamed SDIO
- net SDIO: now also J1.6 (SDIO)
- net RE_B renamed SCLK
- net SCLK: now also J1.1 (SCLK)
- no-connect marks 7 -> 6
